Commit message: added:ScreenShots

File: ur_description/urdf/ur5_arm.urdf.xacro (robot description, xacro)
@@ -21,16 +21,15 @@
     <origin xyz="0.0 0.0 0.0" rpy="0.0 0.0 0.0" />
   </joint>
-  <!-- <joint name="realsense_joint" type="fixed">
+  <joint name="realsense_joint" type="fixed">
     <parent link="wrist_3_link" />
     <child link="camera_link" />
     <origin xyz="0.0 0.0 -0.07" rpy="3.14 0 1.57" />
   </joint>
-  camera in arm configuration
-   -->
-   <joint name="realsense_joint" type="fixed">
+  <!-- camera on arm configuration -->
+   <!-- <joint name="realsense_joint" type="fixed">
     <parent link="base_link" />
     <child link="camera_link" />
     <origin xyz="0.2 0.0 0.7" rpy="0.0 1.2 0.0" />
-  </joint>
+  </joint> -->
   <!-- global camera configuration -->
   <link name="camera_link">

File: ur_description/urdf/ur5_robot.urdf.xacro (robot description, xacro)
@@ -20,16 +20,15 @@
   />
   <link name="world" />
-  <joint name="world_joint" type="fixed">
+  <!-- <joint name="world_joint" type="fixed">
     <parent link="world" />
     <child link = "base_link" />
     <origin xyz="0.0 0.0 0.0" rpy="0.0 0.0 0.0" />
-  </joint>
-   <!-- <joint name="realsense_joint" type="fixed">
+  </joint> -->
+   <joint name="realsense_joint" type="fixed">
     <parent link="wrist_3_link" />
     <child link="camera_link" />
     <origin xyz="0.0 0.0 -0.07" rpy="3.14 0 1.57" />
   </joint>
-  camera in arm configuration
-   -->
+  <!-- camera on arm configuration -->
    <joint name="realsense_joint" type="fixed">
     <parent link="base_link" />
