Commit message: added:new model

File: ur_description/urdf/common.gazebo.xacro (robot description, xacro)
@@ -1,8 +1,3 @@
 <?xml version="1.0"?>
 <robot xmlns:xacro="http://wiki.ros.org/xacro">
-  <gazebo>
-    <plugin name="gazebo_ros2_control" filename="libgazebo_ros2_control.so">
-    <parameters>$(find ur_description)/config/ros_controllers.yaml</parameters>
-    </plugin>
-  </gazebo>
 </robot>

File: ur_description/urdf/realsense2.urdf.xacro (robot description, xacro)
@@ -84,5 +84,5 @@
                 <always_on>1</always_on>
                 <update_rate>30</update_rate>
-                <visualize>0</visualize>
+                <visualize>1</visualize>
             </sensor>
             <sensor name="cameracolor" type="camera">
@@ -106,5 +106,5 @@
                 <always_on>1</always_on>
                 <update_rate>30</update_rate>
-                <visualize>0</visualize>
+                <visualize>1</visualize>
             </sensor>
             <sensor name="cameraired1" type="camera">
@@ -128,5 +128,5 @@
                 <always_on>1</always_on>
                 <update_rate>1</update_rate>
-                <visualize>0</visualize>
+                <visualize>1</visualize>
             </sensor>
             <sensor name="cameraired2" type="camera">
@@ -150,5 +150,5 @@
                 <always_on>1</always_on>
                 <update_rate>1</update_rate>
-                <visualize>0</visualize>
+                <visualize>1</visualize>
             </sensor>
   </gazebo>

File: ur_description/urdf/ur5_arm.urdf.xacro (robot description, xacro)
@@ -11,5 +11,4 @@
   <xacro:include filename="$(find ur_description)/urdf/ur5.urdf.xacro" />
   <xacro:include filename="$(find ur_description)/urdf/realsense2.urdf.xacro" />
-  <!-- arm -->
   <xacro:ur5_robot prefix="" joint_limited="false"
     transmission_hw_interface="$(arg transmission_hw_interface)"
@@ -21,5 +20,5 @@
     <origin xyz="0.0 0.0 0.0" rpy="0.0 0.0 0.0" />
   </joint>
-  <joint name="realsense_joint" type="fixed">
+   <joint name="realsense_joint" type="fixed">
     <parent link="wrist_3_link" />
     <child link="camera_link" />

File: ur_description/urdf/ur5_robot.urdf.xacro (robot description, xacro)
@@ -15,8 +15,10 @@
   <xacro:include filename="$(find ur_description)/urdf/ur5.urdf.xacro" />
   <xacro:include filename="$(find ur_description)/urdf/realsense2.urdf.xacro" />
+  <xacro:include filename="$(find ebot_description)/models/ebot/ebot.gazebo" />
   <!-- arm -->
   <xacro:ur5_robot prefix="" joint_limited="false"
     transmission_hw_interface="$(arg transmission_hw_interface)"
   />
+  <!-- <link name="ebotBaseTop" /> -->
   <link name="world" />
   <!-- <joint name="world_joint" type="fixed">
@@ -31,9 +33,9 @@
   </joint>
   <!-- camera on arm configuration -->
-   <joint name="realsense_joint" type="fixed">
+   <!-- <joint name="realsense_joint" type="fixed">
     <parent link="base_link" />
     <child link="camera_link" />
     <origin xyz="0.2 0.0 0.7" rpy="0.0 1.2 0.0" />
-  </joint>
+  </joint> -->
   <!-- global camera configuration -->
   <link name="camera_link">
