Commit message: added :model added : ur5 ,eye on hand and eye to hand config

File: ur_description/urdf/realsense2.urdf.xacro (robot description, xacro)
@@ -84,5 +84,5 @@
                 <always_on>1</always_on>
                 <update_rate>30</update_rate>
-                <visualize>0</visualize>
+                <visualize>1</visualize>
             </sensor>
             <sensor name="cameracolor" type="camera">
@@ -106,5 +106,5 @@
                 <always_on>1</always_on>
                 <update_rate>30</update_rate>
-                <visualize>0</visualize>
+                <visualize>1</visualize>
             </sensor>
             <sensor name="cameraired1" type="camera">
@@ -128,5 +128,5 @@
                 <always_on>1</always_on>
                 <update_rate>1</update_rate>
-                <visualize>0</visualize>
+                <visualize>1</visualize>
             </sensor>
             <sensor name="cameraired2" type="camera">
@@ -150,5 +150,5 @@
                 <always_on>1</always_on>
                 <update_rate>1</update_rate>
-                <visualize>0</visualize>
+                <visualize>1</visualize>
             </sensor>
   </gazebo>

File: ur_description/urdf/ur5_arm.urdf.xacro (robot description, xacro)
@@ -21,9 +21,17 @@
     <origin xyz="0.0 0.0 0.0" rpy="0.0 0.0 0.0" />
   </joint>
-  <joint name="realsense_joint" type="fixed">
+  <!-- <joint name="realsense_joint" type="fixed">
+    <parent link="wrist_3_link" />
+    <child link="camera_link" />
+    <origin xyz="0.0 0.0 -0.07" rpy="3.14 0 1.57" />
+  </joint>
+  camera in arm configuration
+   -->
+   <joint name="realsense_joint" type="fixed">
     <parent link="base_link" />
     <child link="camera_link" />
     <origin xyz="0.2 0.0 0.7" rpy="0.0 1.2 0.0" />
   </joint>
+  <!-- global camera configuration -->
   <link name="camera_link">
   <collision>

File: ur_description/urdf/ur5_robot.urdf.xacro (robot description, xacro)
@@ -25,9 +25,17 @@
     <origin xyz="0.0 0.0 0.0" rpy="0.0 0.0 0.0" />
   </joint>
-  <joint name="realsense_joint" type="fixed">
+   <!-- <joint name="realsense_joint" type="fixed">
+    <parent link="wrist_3_link" />
+    <child link="camera_link" />
+    <origin xyz="0.0 0.0 -0.07" rpy="3.14 0 1.57" />
+  </joint>
+  camera in arm configuration
+   -->
+   <joint name="realsense_joint" type="fixed">
     <parent link="base_link" />
     <child link="camera_link" />
-    <origin xyz="-0.97 0.0 1.04" rpy="0.0 0.261 0.0" />
+    <origin xyz="0.2 0.0 0.7" rpy="0.0 1.2 0.0" />
   </joint>
+  <!-- global camera configuration -->
   <link name="camera_link">
   <collision>

Commit message: added mesh service

File: ur_description/urdf/realsense2.urdf.xacro (robot description, xacro)
@@ -84,5 +84,5 @@
                 <always_on>1</always_on>
                 <update_rate>30</update_rate>
-                <visualize>1</visualize>
+                <visualize>0</visualize>
             </sensor>
             <sensor name="cameracolor" type="camera">
@@ -106,5 +106,5 @@
                 <always_on>1</always_on>
                 <update_rate>30</update_rate>
-                <visualize>1</visualize>
+                <visualize>0</visualize>
             </sensor>
             <sensor name="cameraired1" type="camera">
@@ -128,5 +128,5 @@
                 <always_on>1</always_on>
                 <update_rate>1</update_rate>
-                <visualize>1</visualize>
+                <visualize>0</visualize>
             </sensor>
             <sensor name="cameraired2" type="camera">
@@ -150,5 +150,5 @@
                 <always_on>1</always_on>
                 <update_rate>1</update_rate>
-                <visualize>1</visualize>
+                <visualize>0</visualize>
             </sensor>
   </gazebo>

File: ur_description/urdf/ur5.urdf.xacro (robot description, xacro)
@@ -24,10 +24,10 @@
     <!-- Inertia parameters -->
     <xacro:property name="base_mass" value="4.0" />  <!-- This mass might be incorrect -->
-    <xacro:property name="shoulder_mass" value="3.7000" />
-    <xacro:property name="upper_arm_mass" value="8.3930" />
-    <xacro:property name="forearm_mass" value="2.2750" />
-    <xacro:property name="wrist_1_mass" value="1.2190" />
-    <xacro:property name="wrist_2_mass" value="1.2190" />
-    <xacro:property name="wrist_3_mass" value="0.1879" />
+    <xacro:property name="shoulder_mass" value="0.01" />
+    <xacro:property name="upper_arm_mass" value="0.01" />
+    <xacro:property name="forearm_mass" value="0.01" />
+    <xacro:property name="wrist_1_mass" value="0.01" />
+    <xacro:property name="wrist_2_mass" value="0.01" />
+    <xacro:property name="wrist_3_mass" value="0.0" />
     <xacro:property name="shoulder_cog" value="0.0 0.00193 -0.02561" />
     <xacro:property name="upper_arm_cog" value="0.0 -0.024201 0.2125" />
